Commit message: added collisions to basic arm urdf

File: src/ainex_arm/urdf/basic_arm.urdf (robot description, URDF)
Before this commit: robot basic_arm, 16 links, 15 joints
Links:
- link Shoulder_servo: geometry collision cylinder length=0.05 radius=0.08; visual cylinder length=0.05 radius=0.08
- link base_servo: geometry collision cylinder length=0.05 radius=0.08; visual cylinder length=0.05 radius=0.08
- link elbow_servo: geometry collision cylinder length=0.05 radius=0.08; visual cylinder length=0.05 radius=0.08
- link right_base_servo: geometry collision cylinder length=0.05 radius=0.08; visual cylinder length=0.05 radius=0.08
- link right_elbow_servo: geometry collision cylinder length=0.05 radius=0.08; visual cylinder length=0.05 radius=0.08
- link right_shoulder_servo: geometry collision cylinder length=0.05 radius=0.08; visual cylinder length=0.05 radius=0.08
