Commit message: sheets updated

File: src/ainex_arm/urdf/robot.urdf (robot description, URDF)
Before this commit: robot basic_arm, 16 links, 15 joints
Links:
- link base_link: mass None -> 2.0; geometry collision box size=0.2 0.3 0.4; visual box size=0.2 0.3 0.4
- link base_servo: mass None -> 0.2; geometry collision sphere radius=0.03; visual sphere radius=0.03
- link elbow_link: mass None -> 0.4; geometry collision box size=0.05 0.2 0.06; visual box size=0.05 0.2 0.06
- link elbow_servo: mass None -> 0.15; geometry collision cylinder length=0.02 radius=0.03; visual cylinder length=0.02 radius=0.03
- link head_link: mass None -> 0.5; geometry collision sphere radius=0.08; visual sphere radius=0.1
- link left_leg_link: mass None -> 0.4; geometry collision box size=0.1 0.1 0.3; visual box size=0.1 0.1 0.3
- link right_base_servo: mass None -> 0.2; geometry collision sphere radius=0.03; visual sphere radius=0.03
- link right_elbow_link: mass None -> 0.4; geometry collision box size=0.05 0.2 0.06; visual box size=0.05 0.2 0.06
- link right_elbow_servo: mass None -> 0.15; geometry collision cylinder length=0.02 radius=0.03; visual cylinder length=0.02 radius=0.03
- link right_leg_link: mass None -> 0.4; geometry collision box size=0.1 0.1 0.3; visual box size=0.1 0.1 0.3
- link right_shoulder_link: mass None -> 0.3; geometry collision box size=0.1 0.1 0.1; visual box size=0.1 0.1 0.1
- link right_shoulder_servo: mass None -> 0.2; geometry collision sphere radius=0.03; visual sphere radius=0.03
- link right_wrist_link: mass None -> 0.3; geometry collision box size=0.1 0.3 0.04; visual box size=0.1 0.3 0.04
- link shoulder_link: mass None -> 0.3; geometry collision box size=0.1 0.1 0.1; visual box size=0.1 0.1 0.1
- link shoulder_servo: mass None -> 0.2; geometry collision sphere radius=0.03; visual sphere radius=0.03
- link wrist_link: mass None -> 0.3; geometry collision box size=0.1 0.3 0.04; visual box size=0.1 0.3 0.04

Commit message: urdf collisions and inertial tags

File: src/ainex_arm/urdf/robot.urdf (robot description, URDF)
Before this commit: robot basic_arm, 16 links, 15 joints
Links:
- link head_link: geometry collision sphere radius=0.1; visual sphere radius=0.1
